File: garden_circ.sch (EAGLE design)
At the start: 39 parts, among them IC1 MEGA8-P, IC2 74HC595N, IC3 74HC595N, IC4 7805TV, J1 POWER_JACKSLT

Commit message: Fixed shift register wiring
Parts:
- added R7: 10K, resistor:R-EU_0207/7
Connections:
- removed net N$38: IC1.PD2(INT0), IC2A.SCL, IC3A.SCL
- new net N$52: IC1.PD2(INT0), IC2A.RCK, IC3A.RCK
- net GND: now also IC2A.SCL, IC3A.SCL; no longer IC2A.RCK, IC3A.RCK
- net N$10: now also R7.2
- net VCC: now also IC1.AREF, R7.1
Changed lines of the file:
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@@
 <part name="GND14" library="supply1" deviceset="GND" device=""/>
 <part name="P+7" library="supply1" deviceset="VCC" device=""/>
-<part name="GND15" library="supply1" deviceset="GND" device=""/>
-<part name="GND16" library="supply1" deviceset="GND" device=""/>
 <part name="JP1" library="pinhead" deviceset="PINHD-2X4" device=""/>
 <part name="P+6" library="supply1" deviceset="VCC" device=""/>
 <part name="X4" library="con-wago-500" deviceset="W237-4" device=""/>
 <part name="J1" library="SparkFun-Connectors" deviceset="POWER_JACK" device="SLT"/>
+<part name="P+8" library="supply1" deviceset="VCC" device=""/>
+<part name="R7" library="resistor" deviceset="R-EU_" device="0207/7" value="10K"/>
 </parts>
 <sheets>
@@
 <instance part="GND14" gate="1" x="-22.86" y="71.12"/>
 <instance part="P+7" gate="VCC" x="-22.86" y="88.9"/>
-<instance part="GND15" gate="1" x="106.68" y="30.48" rot="R270"/>
-<instance part="GND16" gate="1" x="88.9" y="15.24" rot="R180"/>
 <instance part="JP1" gate="A" x="160.02" y="71.12"/>
 <instance part="P+6" gate="VCC" x="172.72" y="81.28"/>
@@
 <instance part="X4" gate="-4" x="-5.08" y="-15.24" rot="R270"/>
 <instance part="J1" gate="G$1" x="-30.48" y="10.16"/>
+<instance part="P+8" gate="VCC" x="5.08" y="104.14"/>
+<instance part="R7" gate="G$1" x="10.16" y="96.52"/>
 </instances>
 <busses>
@@
 <pinref part="IC2" gate="A" pin="G"/>
 <pinref part="GND10" gate="1" pin="GND"/>
+<pinref part="IC2" gate="A" pin="SCL"/>
+<wire x1="109.22" y1="35.56" x2="106.68" y2="35.56" width="0.1524" layer="91"/>
+<wire x1="106.68" y1="35.56" x2="106.68" y2="20.32" width="0.1524" layer="91"/>
+<wire x1="106.68" y1="20.32" x2="109.22" y2="20.32" width="0.1524" layer="91"/>
 </segment>
 <segment>
 <pinref part="IC3" gate="A" pin="G"/>
 <pinref part="GND9" gate="1" pin="GND"/>
+<pinref part="IC3" gate="A" pin="SCL"/>
+<wire x1="93.98" y1="10.16" x2="93.98" y2="15.24" width="0.1524" layer="91"/>
+<wire x1="93.98" y1="15.24" x2="83.82" y2="15.24" width="0.1524" layer="91"/>
+<wire x1="83.82" y1="15.24" x2="83.82" y2="10.16" width="0.1524" layer="91"/>
+<wire x1="83.82" y1="10.16" x2="78.74" y2="10.16" width="0.1524" layer="91"/>
+<junction x="78.74" y="10.16"/>
 </segment>
 <segment>
@@
 <junction x="-43.18" y="76.2"/>
 <pinref part="GND14" gate="1" pin="GND"/>
-</segment>
-<segment>
-<pinref part="IC2" gate="A" pin="RCK"/>
-<pinref part="GND15" gate="1" pin="GND"/>
-</segment>
-<segment>
-<pinref part="IC3" gate="A" pin="RCK"/>
-<pinref part="GND16" gate="1" pin="GND"/>
-<wire x1="88.9" y1="12.7" x2="88.9" y2="10.16" width="0.1524" layer="91"/>
 </segment>
 </net>
@@
 </segment>
 </net>
-<net name="N$38" class="0">
-<segment>
-<pinref part="IC1" gate="G$1" pin="PD2(INT0)"/>
-<wire x1="63.5" y1="58.42" x2="104.14" y2="58.42" width="0.1524" layer="91"/>
-<wire x1="104.14" y1="58.42" x2="104.14" y2="35.56" width="0.1524" layer="91"/>
-<pinref part="IC2" gate="A" pin="SCL"/>
-<wire x1="104.14" y1="35.56" x2="109.22" y2="35.56" width="0.1524" layer="91"/>
-<pinref part="IC3" gate="A" pin="SCL"/>
-<wire x1="93.98" y1="10.16" x2="93.98" y2="35.56" width="0.1524" layer="91"/>
-<wire x1="93.98" y1="35.56" x2="104.14" y2="35.56" width="0.1524" layer="91"/>
-<junction x="104.14" y="35.56"/>
-</segment>
-</net>
 <net name="N$9" class="0">
 <segment>
@@
 <wire x1="134.62" y1="71.12" x2="134.62" y2="96.52" width="0.1524" layer="91"/>
 <wire x1="134.62" y1="96.52" x2="15.24" y2="96.52" width="0.1524" layer="91"/>
+<pinref part="R7" gate="G$1" pin="2"/>
+<junction x="15.24" y="96.52"/>
 </segment>
 </net>
@@
 <wire x1="12.7" y1="40.64" x2="15.24" y2="40.64" width="0.1524" layer="91"/>
 <junction x="15.24" y="40.64"/>
+<pinref part="IC1" gate="G$1" pin="AREF"/>
+<wire x1="15.24" y1="78.74" x2="12.7" y2="78.74" width="0.1524" layer="91"/>
+<wire x1="12.7" y1="78.74" x2="12.7" y2="76.2" width="0.1524" layer="91"/>
+<junction x="12.7" y="76.2"/>
 </segment>
 <segment>
@@
 <junction x="-5.08" y="-20.32"/>
 </segment>
+<segment>
+<pinref part="P+8" gate="VCC" pin="VCC"/>
+<wire x1="5.08" y1="101.6" x2="5.08" y2="96.52" width="0.1524" layer="91"/>
+<pinref part="R7" gate="G$1" pin="1"/>
+</segment>
 </net>
 <net name="N$19" class="0">
@@
 </segment>
 </net>
+<net name="N$52" class="0">
+<segment>
+<pinref part="IC3" gate="A" pin="RCK"/>
+<wire x1="88.9" y1="12.7" x2="88.9" y2="10.16" width="0.1524" layer="91"/>
+<wire x1="88.9" y1="12.7" x2="104.14" y2="12.7" width="0.1524" layer="91"/>
+<pinref part="IC1" gate="G$1" pin="PD2(INT0)"/>
+<wire x1="63.5" y1="58.42" x2="104.14" y2="58.42" width="0.1524" layer="91"/>
+<wire x1="104.14" y1="58.42" x2="104.14" y2="30.48" width="0.1524" layer="91"/>
+<pinref part="IC2" gate="A" pin="RCK"/>
+<wire x1="104.14" y1="30.48" x2="109.22" y2="30.48" width="0.1524" layer="91"/>
+<wire x1="104.14" y1="12.7" x2="104.14" y2="30.48" width="0.1524" layer="91"/>
+<junction x="104.14" y="30.48"/>
+</segment>
+</net>
