File: garden_circ.sch (EAGLE design)
At the start: 47 parts, among them IC1 MEGA8-P, IC2 74HC595D, IC3 74HC595D, IC4 7805DT, J1 POWER_JACKSLT, Q3 MOSFET-NCHANNELBSS123LT1G

Commit message: Added a few tweaks and power light
Parts:
- added H3, H4: MOUNT-HOLE2.8, holes:MOUNT-HOLE2.8
- added JP1: (no value), pinhead:PINHD-1X4
- added LED7: (no value), led:LEDSML0805
- added R19: 220, SparkFun-Resistors:RESISTOR0805-RES
- added S1, S2, S3: SWITCH-MOMENTARY-2PTH, SparkFun-Electromechanical:SWITCH-MOMENTARY-2PTH
Connections:
- new net N$69: IC3A.QC, R18.2
- new net N$70: JP1.2, S2.1
- new net N$71: JP1.3, S1.1
- new net N$72: JP1.4, S1.2, S2.2, S3.2
- new net N$73: LED7.C, R19.2
- net GND: now also JP4.5, R19.1, R8.A; no longer JP4.16
- net N$66: now also JP1.1, S3.1; no longer Q3.D, R8.A
- net N$67: now also JP4.16, Q3.D; no longer IC2A.QH, R18.2
- net VCC: now also LED7.A
Other:
- moved on the sheet: JP4, Q3, R18, X1-3, X1-4, X1-5
