File: old/garden_circ.sch (EAGLE design)
At the start: 47 parts, among them IC1 MEGA8-P, IC2 74HC595D, IC3 74HC595D, IC4 7805DT, J1 POWER_JACKSLT, Q3 MOSFET-NCHANNELBSS123LT1G

Commit message: Added code an SMD board
Parts:
- removed H1, H2: MOUNT-HOLE2.8, holes:MOUNT-HOLE2.8
- removed JP2: (no value), pinhead:PINHD-2X3
- removed JP3: (no value), pinhead:PINHD-1X2
- removed JP4: (no value), pinhead:PINHD-1X16
- removed JP5: (no value), pinhead:PINHD-1X4
- removed Q3: MOSFET-NCHANNELBSS123LT1G, SparkFun-DiscreteSemi:MOSFET-NCHANNELBSS123LT1G
- removed R18: (no value), SparkFun-Resistors:RESISTOR0805-RES
- removed R8: (no value), resistor:R-TRIMM3202
- added JP1: (no value), pinhead:PINHD-2X4
- added SV1: (no value), con-lstb:MA20-1
- C1, C2, C5, C6, C7: device SparkFun-Capacitors:CAP0805 -> rcl:C-EU025-040X050
- C3, C4: device resistor:CPOL-EUSMCC -> resistor:CPOL-EUE2.5-5
- IC2, IC3: value 74HC595D -> 74HC595N; device 74xx-eu:74HC595D -> 74xx-eu:74HC595N
- IC4: value 7805DT -> 7805TV; device linear:7805DT -> linear:7805TV
- Q1: device crystal:CRYSTALHC49UP -> crystal:CRYSTALHC49U-V
- R1, R10, R11, R12, R13, R14, R15, R16, R17, R2, R3, R4, R5, R6, R9: device SparkFun-Resistors:RESISTOR0805-RES -> rcl:R-EU_0204/7
- R7: device SparkFun-Resistors:RESISTOR0805-RES -> resistor:R-EU_0207/7
Connections:
- removed net MISO: IC1.PB4(MISO), JP2.1
- removed net N$59: JP4.3, R8.S
- removed net N$65: IC3A.QE, JP4.11
- removed net N$66: Q3.D, R8.A
- removed net N$67: IC2A.QH, R18.2
- removed net N$68: Q3.G, R18.1
- net GND: now also JP1.6, SV1.1, SV1.14, SV1.17, X1-6.KL; no longer JP2.6, JP4.1, JP4.16, JP5.4, Q3.S
- net N$10: now also JP1.5; no longer JP2.5
- net N$19: now also JP1.8; no longer JP3.2
- net N$20: now also JP1.3; no longer JP2.3
- net N$26: now also SV1.9; no longer JP4.6
- net N$27: now also SV1.4; no longer JP4.4
- net N$28: now also IC3A.QE, SV1.10; no longer IC3A.QH, JP4.14
- net N$29: now also IC3A.QF, SV1.11; no longer IC3A.QG, JP4.13
- net N$30: now also IC3A.QG, SV1.12; no longer IC3A.QF, JP4.12
- net N$39: now also SV1.18; no longer JP5.1
- net N$40: now also SV1.19; no longer JP5.2
- net N$41: now also SV1.20; no longer JP5.3
- net N$44: now also JP1.4; no longer JP2.4
- net N$45: now also JP1.7; no longer JP3.1
- net N$9: now also IC1.PB4(MISO), JP1.1; no longer IC2A.QG, X1-6.KL
- net VCC: now also JP1.2, SV1.13, SV1.2; no longer JP2.2, JP4.15, JP4.2, R8.E
Other:
- moved on the sheet: C1, C2, C5, C6, C7, IC3, X1-6
